File: pcb/corne-cherry.kicad_pcb (KiCad board)
At the start: 2 copper layers, 275.5 x 105.6 mm, 176 parts, among them J1 MJ-4PP-9, J2 OLED, J3 MJ-4PP-9, J4 OLED, J5 Conn_01x01_Male, J6 Conn_01x01_Male, P1 Conn_01x03, P3 Conn_01x03, SW1 SW_PUSH, SW10 SW_PUSH, SW11 SW_PUSH, SW12 SW_PUSH, SW13 SW_PUSH, SW14 SW_PUSH, SW15 SW_PUSH, SW16 SW_PUSH, SW17 SW_PUSH, SW18 SW_PUSH, SW19 SW_PUSH, SW2 SW_PUSH, SW20 SW_PUSH, SW21 SW_PUSH, SW22 SW_PUSH, SW23 SW_PUSH, SW24 SW_PUSH, SW25 SW_PUSH, SW26 SW_PUSH, SW27 SW_PUSH, SW28 SW_PUSH, SW29 SW_PUSH, SW3 SW_PUSH, SW30 SW_PUSH, SW31 SW_PUSH, SW32 SW_PUSH, SW33 SW_PUSH, SW34 SW_PUSH, SW35 SW_PUSH, SW36 SW_PUSH, SW37 SW_PUSH, SW38 SW_PUSH, SW39 SW_PUSH, SW4 SW_PUSH, SW40 SW_PUSH, SW41 SW_PUSH, SW42 SW_PUSH, SW43 Rotary_Encoder_Switch, SW44 Rotary_Encoder_Switch, SW5 SW_PUSH, SW6 SW_PUSH, SW7 SW_PUSH, SW8 SW_PUSH, SW9 SW_PUSH, U1 ProMicro, U2 ProMicro

Commit message: removed the weeb stuff to make a nice and clean pcb and regenreated gerbers
Parts:
- removed the G*** at (160.9, 43.5)
- removed the G*** at (133.7, 43.6)
- removed the G*** at (265.3, 58.7)
- removed the G*** at (32.7, 64.1)
- removed the G*** at (69.4, 77.0)
- removed the G*** at (221.0, 76.8)
Other:
- board text removed: "https://github.com/ItsWaffIe/waffIe_corne"
- board text removed: "https://github.com/foostan/crkbd"
